Commit message: Document IMU setup in simple URDF

File: src/bumperbot_description/urdf/bumperbot_gazebo.xacro (robot description, xacro)
@@ -55,3 +55,72 @@
     <maxVel>0.1</maxVel>
   </gazebo>
+  <!-- ROS 2 Control -->
+<gazebo>
+  <!-- ROS 2 Humble (Ignition) -->
+  <xacro:if value="${arg is_ignition}">
+    <plugin filename="ign_ros2_control-system" name="ign_ros2_control::IgnitionROS2ControlPlugin">
+      <parameters>$(find bumperbot_controller)/config/bumperbot_controllers.yaml</parameters>
+    </plugin>
+    <plugin filename="ignition-gazebo-imu-system" name="ignition::gazebo::systems::Imu"/>
+  </xacro:if>
+  <!-- ROS 2 Iron or above (Gazebo / ros_gz_sim) -->
+  <xacro:unless value="${arg is_ignition}">
+    <plugin filename="gz_ros2_control-system" name="gz_ros2_control::GazeboSimROS2ControlPlugin">
+      <parameters>$(find bumperbot_controller)/config/bumperbot_controllers.yaml</parameters>
+    </plugin>
+    <plugin filename="gz-sim-imu-system" name="gz::sim::systems::Imu"/>
+  </xacro:unless>
+</gazebo>
+<gazebo reference="imu_link">
+  <sensor name="imu" type="imu">
+    <always_on>true</always_on>
+    <update_rate>100</update_rate>
+    <gz_frame_id>imu_link</gz_frame_id>
+    <topic>imu</topic>
+    <imu>
+      <!-- Angular velocity noise -->
+      <angular_velocity>
+        <x>
+          <noise type="gaussian">
+            <mean>0.0</mean>
+            <stddev>2e-4</stddev>
+          </noise>
+        </x>
+        <y>
+          <noise type="gaussian">
+            <mean>0.0</mean>
+            <stddev>2e-4</stddev>
+          </noise>
+        </y>
+        <z>
+          <noise type="gaussian">
+            <mean>0.0</mean>
+            <stddev>2e-4</stddev>
+          </noise>
+        </z>
+      </angular_velocity>
+      <!-- Linear acceleration noise -->
+      <linear_acceleration>
+        <x>
+          <noise type="gaussian">
+            <mean>0.0</mean>
+            <stddev>1.7e-2</stddev>
+          </noise>
+        </x>
+        <y>
+          <noise type="gaussian">
+            <mean>0.0</mean>
+            <stddev>1.7e-2</stddev>
+          </noise>
+        </y>
+        <z>
+          <noise type="gaussian">
+            <mean>0.0</mean>
+            <stddev>1.7e-2</stddev>
+          </noise>
+        </z>
+      </linear_acceleration>
+    </imu>
+  </sensor>
+</gazebo>
 </xacro:macro>

File: src/bumperbot_description/urdf/bumperbot_simple.urdf.xacro (robot description, xacro)
@@ -1,10 +1,20 @@
 <?xml version="1.0"?>
-<!-- Minimal bumperbot with two drive wheels and ros2_control mock hardware. -->
+<!--
+  Minimal bumperbot model used by gazebo_simple_control.launch.py.
+  The intent is to keep geometry lightweight while still exercising ros2_control,
+  wheel kinematics, and an IMU pipeline for testing controllers and filters.
+-->
 <robot name="bumperbot" xmlns:xacro="http://ros.org/wiki/xacro">
+  <!-- Runtime arguments so the same URDF can tweak the IMU plugin without editing the file. -->
+  <xacro:arg name="imu_plugin_filename" default="libgazebo_ros_imu_sensor.so"/>
+  <xacro:arg name="imu_topic" default="imu"/>
   <!-- Base footprint (map->base_footprint->base_link) -->
+  <!-- Thin link used so TF trees can attach map/odom frames cleanly in localization stacks. -->
   <link name="base_footprint"/>
   <!-- Main chassis -->
+  <!-- Box body keeps inertial math simple while roughly matching the real bumperbot volume. -->
   <link name="base_link">
     <inertial>
+      <!-- Center of mass located slightly above the ground plane to reflect chassis height. -->
       <origin xyz="0 0 0.04" rpy="0 0 0" />
       <mass value="0.8"/>
@@ -12,4 +22,5 @@
     </inertial>
     <visual>
+      <!-- Simple box visual keeps Gazebo rendering cheap. -->
       <origin xyz="0 0 0.04" rpy="0 0 0" />
       <geometry>
@@ -19,4 +30,5 @@
     </visual>
     <collision>
+      <!-- Reuse the box for collision; matches wheel height so contact behaves well. -->
       <origin xyz="0 0 0.04" rpy="0 0 0" />
       <geometry>
@@ -26,4 +38,5 @@
   </link>
   <!-- Fixed transform from base_footprint to base_link -->
+  <!-- Keeps the chassis floating 3.3 cm above the footprint plane. -->
   <joint name="base_joint" type="fixed">
     <parent link="base_footprint"/>
@@ -32,4 +45,5 @@
   </joint>
   <!-- Right wheel as a cylinder -->
+  <!-- Cylindrical wheels are sufficient for differential-drive kinematics and collisions. -->
   <link name="wheel_right_link">
     <visual>
@@ -40,9 +54,11 @@
     </visual>
     <collision>
-      <geometry>
-        <cylinder radius="0.033" length="0.02"/>
-      </geometry>
-    </collision>
-    <inertial>
+      <!-- Match the visual geometry so contact forces line up with the mesh. -->
+      <geometry>
+        <cylinder radius="0.033" length="0.02"/>
+      </geometry>
+    </collision>
+    <inertial>
+      <!-- Lightweight wheels so acceleration behaves realistically in simulation. -->
       <mass value="0.05"/>
       <inertia ixx="0.0001" ixy="0" ixz="0" iyy="0.0001" iyz="0" izz="0.0001"/>
@@ -50,4 +66,5 @@
   </link>
   <joint name="wheel_right_joint" type="continuous">
+    <!-- Position wheel on the negative Y side; roll axis aligns with Gazebo convention. -->
     <origin xyz="0 -0.07 0" rpy="1.57 0 0" />
     <parent link="base_link" />
@@ -56,4 +73,5 @@
   </joint>
   <!-- Gazebo contact/friction for right wheel to ensure traction -->
+  <!-- High mu values prevent sliding so velocity controllers have predictable behavior. -->
   <gazebo reference="wheel_right_link">
     <mu1>1.0</mu1>
@@ -84,4 +102,5 @@
   </link>
   <joint name="wheel_left_joint" type="continuous">
+    <!-- Mirror of the right wheel: positive Y offset, same axle orientation. -->
     <origin xyz="0 0.07 0" rpy="1.57 0 0" />
     <parent link="base_link" />
@@ -99,5 +118,99 @@
     <fdir1>1 0 0</fdir1>
   </gazebo>
+  <!-- IMU link for sensor frame alignment -->
+  <!-- Bring over the detailed inertial properties so filters can model the IMU accurately. -->
+  <link name="imu_link">
+    <inertial>
+      <origin xyz="-0.00552433659106688 0.000168210391520346 0.000514000497342681" rpy="0 0 0" />
+      <mass value="0.000528415362211671" />
+      <inertia ixx="1.46176048428261E-08" ixy="1.40015117949421E-10" ixz="-1.99633872937403E-12"
+               iyy="8.59662482954888E-09" iyz="7.52375112767959E-12"
+               izz="2.30279421279312E-08" />
+    </inertial>
+    <visual>
+      <!-- Reference an STL so the sensor appears in RViz/Gazebo for debugging. -->
+      <origin xyz="0 0 0" rpy="0 0 0" />
+      <geometry>
+        <mesh filename="package://bumperbot_description/meshes/imu_link.STL" />
+      </geometry>
+      <material name="imu_gray">
+        <color rgba="0.792156862745098 0.819607843137255 0.933333333333333 1" />
+      </material>
+    </visual>
+    <collision>
+      <!-- Use the same mesh for collision to catch accidental contacts in sim. -->
+      <origin xyz="0 0 0" rpy="0 0 0" />
+      <geometry>
+        <mesh filename="package://bumperbot_description/meshes/imu_link.STL" />
+      </geometry>
+    </collision>
+  </link>
+  <joint name="imu_joint" type="fixed">
+    <!-- Mount the IMU above the chassis center for realistic sensor frame alignment. -->
+    <origin xyz="0 0 0.0698986241758014" rpy="0 0 0" />
+    <parent link="base_link" />
+    <child link="imu_link" />
+    <axis xyz="0 0 0" />
+  </joint>
+  <!-- Gazebo sensor definition so Classic publishes IMU data with configurable noise. -->
+  <gazebo reference="imu_link">
+    <sensor name="imu" type="imu">
+      <always_on>true</always_on>
+      <update_rate>100</update_rate>
+      <gz_frame_id>imu_link</gz_frame_id>
+      <topic>$(arg imu_topic)</topic>
+      <imu>
+        <angular_velocity>
+          <x>
+            <!-- Gaussian noise per axis keeps angular velocity data realistic. -->
+            <noise type="gaussian">
+              <mean>0.0</mean>
+              <stddev>2e-4</stddev>
+            </noise>
+          </x>
+          <y>
+            <noise type="gaussian">
+              <mean>0.0</mean>
+              <stddev>2e-4</stddev>
+            </noise>
+          </y>
+          <z>
+            <noise type="gaussian">
+              <mean>0.0</mean>
+              <stddev>2e-4</stddev>
+            </noise>
+          </z>
+        </angular_velocity>
+        <linear_acceleration>
+          <x>
+            <!-- Acceleration noise tuned to match consumer-grade IMU specs. -->
+            <noise type="gaussian">
+              <mean>0.0</mean>
+              <stddev>1.7e-2</stddev>
+            </noise>
+          </x>
+          <y>
+            <noise type="gaussian">
+              <mean>0.0</mean>
+              <stddev>1.7e-2</stddev>
+            </noise>
+          </y>
+          <z>
+            <noise type="gaussian">
+              <mean>0.0</mean>
+              <stddev>1.7e-2</stddev>
+            </noise>
+          </z>
+        </linear_acceleration>
+      </imu>
+      <plugin name="imu_plugin" filename="$(arg imu_plugin_filename)">
+        <!-- Classic Gazebo expects these tags instead of ROS 2 remappings. -->
+        <topicName>$(arg imu_topic)</topicName>
+        <frameName>imu_link</frameName>
+      </plugin>
+    </sensor>
+  </gazebo>
   <!-- ros2_control hardware + interfaces for wheel joints (Gazebo integration) -->
+  <!-- Plugin block declares the simulated hardware interface with velocity commands. -->
   <ros2_control name="BumperBotSystem" type="system">
     <hardware>
