Commit message: Add multi_robot_bringup package for two-robot Nav2 simulation
New package launches two bumperbot robots in one Gazebo world with fully
isolated Nav2 stacks using namespaced TF (/robot1/tf, /robot2/tf).

Key changes:
- bumperbot_gazebo.xacro: add is_primary param to prevent Ogre2 segfault
  from duplicate Sensors plugins, add TF remappings for namespace isolation
- bumperbot_controllers.yaml: add /** wildcard + tf_frame_prefix_enable:false
  for multi-robot namespace support
- multi_robot_bringup: complete package with per-robot bringup (controllers,
  AMCL, map_server, full Nav2 stack), staggered timing, costmap topic
  override for correct namespace resolution, and RViz for robot1

Co-Authored-By: Claude Opus 4.6 <noreply@anthropic.com>

File: src/bumperbot_description/urdf/bumperbot_gazebo.xacro (robot description, xacro)
@@ -1,6 +1,9 @@
 <?xml version="1.0"?>
 <robot name="bumperbot" xmlns:xacro="http://ros.org/wiki/xacro">
-  <!-- Macro that injects Gazebo / gz_ros2_control plugins for a namespaced robot -->
-  <xacro:macro name="bumperbot_gazebo" params="ros_namespace">
+  <!-- Macro that injects Gazebo / gz_ros2_control plugins for a namespaced robot.
+       is_primary=true loads world-level singleton system plugins (Sensors, IMU).
+       Set is_primary=false on all but one robot in a multi-robot scene — loading
+       those plugins twice crashes Ogre2 (libGLdispatch segfault). -->
+  <xacro:macro name="bumperbot_gazebo" params="ros_namespace is_primary:=true">
     <!-- Wheels -->
     <gazebo reference="wheel_left_link">
@@ -46,12 +49,18 @@
           <ros>
             <namespace>${ros_namespace}</namespace>
+            <!-- Redirect TF to namespaced topic so each robot owns its TF tree.
+                 When ros_namespace="" (single robot) this resolves to /tf — no change. -->
+            <remapping>/tf:=tf</remapping>
+            <remapping>/tf_static:=tf_static</remapping>
           </ros>
           <parameters>$(find bumperbot_controller)/config/bumperbot_controllers.yaml</parameters>
         </plugin>
-        <plugin filename="ignition-gazebo-imu-system" name="ignition::gazebo::systems::Imu"/>
-        <plugin filename="ignition-gazebo-sensors-system" name="ignition::gazebo::systems::Sensors">
-          <!-- Use Ogre2 rendering so GPU lidar works correctly -->
-          <render_engine>ogre2</render_engine>
-        </plugin>
+        <xacro:if value="${is_primary}">
+          <plugin filename="ignition-gazebo-imu-system" name="ignition::gazebo::systems::Imu"/>
+          <plugin filename="ignition-gazebo-sensors-system" name="ignition::gazebo::systems::Sensors">
+            <!-- Use Ogre2 rendering so GPU lidar works correctly -->
+            <render_engine>ogre2</render_engine>
+          </plugin>
+        </xacro:if>
       </xacro:if>
       <!-- ROS 2 Iron+ / gz_sim path -->
@@ -60,12 +69,16 @@
           <ros>
             <namespace>${ros_namespace}</namespace>
+            <remapping>/tf:=tf</remapping>
+            <remapping>/tf_static:=tf_static</remapping>
           </ros>
           <parameters>$(find bumperbot_controller)/config/bumperbot_controllers.yaml</parameters>
         </plugin>
-        <plugin filename="gz-sim-imu-system" name="gz::sim::systems::Imu"/>
-        <plugin filename="gz-sim-sensors-system" name="gz::sim::systems::Sensors">
-          <!-- Use Ogre2 rendering so GPU lidar works correctly -->
-          <render_engine>ogre2</render_engine>
-        </plugin>
+        <xacro:if value="${is_primary}">
+          <plugin filename="gz-sim-imu-system" name="gz::sim::systems::Imu"/>
+          <plugin filename="gz-sim-sensors-system" name="gz::sim::systems::Sensors">
+            <!-- Use Ogre2 rendering so GPU lidar works correctly -->
+            <render_engine>ogre2</render_engine>
+          </plugin>
+        </xacro:if>
       </xacro:unless>
     </gazebo>
