Commit message: Initial commit: ROS2 bumperbot with working ros2_control
- Added bumperbot_description package with URDF/Xacro files
- Added bumperbot_controller package with working controller config
- Fixed controller configuration (publish_rate as float)
- Working differential drive controller and joint state broadcaster
- Gazebo integration with mock hardware
- Launch files for RViz, Gazebo, and Webots

File: src/bumperbot_description/urdf/bumperbot.urdf.xacro (robot description, xacro)
@@ -1,5 +1,4 @@
 <?xml version="1.0"?>
 <robot name="bumperbot" xmlns:xacro="http://ros.org/wiki/xacro">
-  <xacro:arg name="is_ignition" default="true" />
   <!-- Include Gazebo Parameters -->
   <xacro:include filename="$(find bumperbot_description)/urdf/bumperbot_gazebo.xacro" />
@@ -58,6 +57,5 @@
     <axis xyz="0 1 0" />
   </joint>
-  <link
-    name="wheel_left_link">
+  <link name="wheel_left_link">
     <inertial>
       <origin xyz="0 0.014 0" rpy="0 0 0" />

File: src/bumperbot_description/urdf/bumperbot_gazebo.xacro (robot description, xacro)
@@ -1,5 +1,21 @@
 <?xml version="1.0"?>
-<robot name="bumperbot" xmlns:xacro="http://ros.org/wiki/xacro">
-  <gazebo reference= "Wheel_right_link">
+<robot name="bumperbot" xmlns:xacro="http://www.ros.org/wiki/xacros">
+  <!-- Add material colors for visibility -->
+  <gazebo reference="base_link">
+    <material>Gazebo/Blue</material>
+  </gazebo>
+  <gazebo reference="wheel_right_link">
+    <material>Gazebo/Black</material>
+  </gazebo>
+  <gazebo reference="wheel_left_link">
+    <material>Gazebo/Black</material>
+  </gazebo>
+  <gazebo reference="caster_front_link">
+    <material>Gazebo/Red</material>
+  </gazebo>
+  <gazebo reference="caster_rear_link">
+    <material>Gazebo/Red</material>
+  </gazebo>
+  <gazebo reference="wheel_right_link">
     <mu1>100000000000000.0</mu1>
     <mu2>100000000000000.0</mu2>
@@ -10,5 +26,5 @@
     <fdirl>1 0 0</fdirl>
   </gazebo>
-  <gazebo reference= "Wheel_left_link">
+  <gazebo reference="wheel_left_link">
     <mu1>100000000000000.0</mu1>
     <mu2>100000000000000.0</mu2>
@@ -19,5 +35,5 @@
     <fdirl>1 0 0</fdirl>
   </gazebo>
-  <gazebo reference= "caster_front_link">
+  <gazebo reference="caster_front_link">
     <mu1>0.1</mu1>
     <mu2>0.1</mu2>
@@ -27,5 +43,5 @@
     <maxVel>0.1</maxVel>
   </gazebo>
-  <gazebo reference= "caster_rear_link">
+  <gazebo reference="caster_rear_link">
     <mu1>0.1</mu1>
     <mu2>0.1</mu2>
@@ -35,20 +51,10 @@
     <maxVel>0.1</maxVel>
   </gazebo>
-  <!-- Pick the right ros2_control plugin: Ignition or classic Gazebo -->
+ <!---
   <gazebo>
-    <!-- When launching with ignition-gazebo (ros_gz), use the Ignition plugin -->
-    <xacro:if value="$(arg is_ignition)">
-      <plugin filename="ign_ros2_control-system"
-              name="ign_ros2_control::IgnitionROS2ControlPlugin">
-        <parameters></parameters>
-      </plugin>
-    </xacro:if>
-    <!-- When *not* using ignition (i.e., classic Gazebo), load the gz_ros2_control plugin -->
-    <xacro:unless value="$(arg is_ignition)">
-      <plugin filename="gz_ros2_control-system"
-              name="gz_ros2_control::GazeboSimROS2ControlPlugin">
-        <parameters></parameters>
-      </plugin>
-    </xacro:unless>
+    <plugin name="gazebo_ros_factory" filename="libgazebo_ros_factory.so">
+      <parameters>$(find bumperbot_controller)/config/bumperbot_controllers.yaml</parameters>
+    </plugin>
   </gazebo>
+  -->
 </robot>

Commit message: Import local changes from ZIP working copy

File: src/bumperbot_description/urdf/bumperbot.urdf.xacro (robot description, xacro)
@@ -3,4 +3,5 @@
   <!-- Include Gazebo Parameters -->
   <xacro:include filename="$(find bumperbot_description)/urdf/bumperbot_gazebo.xacro" />
+  <xacro:bumperbot_gazebo_props />
   <link name="base_footprint"/>
   <link name="base_link">

File: src/bumperbot_description/urdf/bumperbot_gazebo.xacro (robot description, xacro)
@@ -1,5 +1,7 @@
 <?xml version="1.0"?>
-<robot name="bumperbot" xmlns:xacro="http://www.ros.org/wiki/xacros">
-  <!-- Add material colors for visibility -->
+<!-- Gazebo-specific visuals and contact/friction parameters.
+     This file is included by xacro; do not wrap in a <robot> tag. -->
+<xacro:macro name="bumperbot_gazebo_props" xmlns:xacro="http://ros.org/wiki/xacro">
+  <!-- Colors for quick visual identification -->
   <gazebo reference="base_link">
     <material>Gazebo/Blue</material>
@@ -17,22 +19,24 @@
     <material>Gazebo/Red</material>
   </gazebo>
+  <!-- High friction on drive wheels to avoid slipping in simple worlds -->
   <gazebo reference="wheel_right_link">
-    <mu1>100000000000000.0</mu1>
-    <mu2>100000000000000.0</mu2>
-    <kp>1000000000000.0</kp>
+    <mu1>1.0</mu1>
+    <mu2>1.0</mu2>
+    <kp>1000000.0</kp>
     <kd>10.0</kd>
     <minDepth>0.001</minDepth>
     <maxVel>0.1</maxVel>
-    <fdirl>1 0 0</fdirl>
+    <fdir1>1 0 0</fdir1>
   </gazebo>
   <gazebo reference="wheel_left_link">
-    <mu1>100000000000000.0</mu1>
-    <mu2>100000000000000.0</mu2>
-    <kp>1000000000000.0</kp>
+    <mu1>1.0</mu1>
+    <mu2>1.0</mu2>
+    <kp>1000000.0</kp>
     <kd>10.0</kd>
     <minDepth>0.001</minDepth>
     <maxVel>0.1</maxVel>
-    <fdirl>1 0 0</fdirl>
+    <fdir1>1 0 0</fdir1>
   </gazebo>
+  <!-- Lower friction on casters so they slide/rotate easily -->
   <gazebo reference="caster_front_link">
     <mu1>0.1</mu1>
@@ -51,10 +55,3 @@
     <maxVel>0.1</maxVel>
   </gazebo>
- <!---
-  <gazebo>
-    <plugin name="gazebo_ros_factory" filename="libgazebo_ros_factory.so">
-      <parameters>$(find bumperbot_controller)/config/bumperbot_controllers.yaml</parameters>
-    </plugin>
-  </gazebo>
-  -->
-</robot>
+</xacro:macro>

Commit message: docs: add comments across launch/YAML/URDF/scripts; add Flask+Socket.IO web UI for cmd_vel; align controller.launch with YAML

File: src/bumperbot_description/urdf/bumperbot.urdf.xacro (robot description, xacro)
@@ -1,7 +1,56 @@
 <?xml version="1.0"?>
 <robot name="bumperbot" xmlns:xacro="http://ros.org/wiki/xacro">
-  <!-- Include Gazebo Parameters -->
-  <xacro:include filename="$(find bumperbot_description)/urdf/bumperbot_gazebo.xacro" />
-  <xacro:bumperbot_gazebo_props />
+  <!-- Gazebo-specific visuals and contact/friction parameters (inlined) -->
+  <gazebo reference="base_link">
+    <material>Gazebo/Blue</material>
+  </gazebo>
+  <gazebo reference="wheel_right_link">
+    <material>Gazebo/Black</material>
+  </gazebo>
+  <gazebo reference="wheel_left_link">
+    <material>Gazebo/Black</material>
+  </gazebo>
+  <gazebo reference="caster_front_link">
+    <material>Gazebo/Red</material>
+  </gazebo>
+  <gazebo reference="caster_rear_link">
+    <material>Gazebo/Red</material>
+  </gazebo>
+  <!-- High friction on drive wheels to avoid slipping in simple worlds -->
+  <gazebo reference="wheel_right_link">
+    <mu1>1.0</mu1>
+    <mu2>1.0</mu2>
+    <kp>1000000.0</kp>
+    <kd>10.0</kd>
+    <minDepth>0.001</minDepth>
+    <maxVel>0.1</maxVel>
+    <fdir1>1 0 0</fdir1>
+  </gazebo>
+  <gazebo reference="wheel_left_link">
+    <mu1>1.0</mu1>
+    <mu2>1.0</mu2>
+    <kp>1000000.0</kp>
+    <kd>10.0</kd>
+    <minDepth>0.001</minDepth>
+    <maxVel>0.1</maxVel>
+    <fdir1>1 0 0</fdir1>
+  </gazebo>
+  <!-- Lower friction on casters so they slide/rotate easily -->
+  <gazebo reference="caster_front_link">
+    <mu1>0.1</mu1>
+    <mu2>0.1</mu2>
+    <kp>1000000.0</kp>
+    <kd>100.0</kd>
+    <minDepth>0.001</minDepth>
+    <maxVel>0.1</maxVel>
+  </gazebo>
+  <gazebo reference="caster_rear_link">
+    <mu1>0.1</mu1>
+    <mu2>0.1</mu2>
+    <kp>1000000.0</kp>
+    <kd>100.0</kd>
+    <minDepth>0.001</minDepth>
+    <maxVel>0.1</maxVel>
+  </gazebo>
   <link name="base_footprint"/>
   <link name="base_link">

File: src/bumperbot_description/urdf/bumperbot_simple.urdf.xacro (robot description, xacro)
@@ -1,5 +1,8 @@
 <?xml version="1.0"?>
+<!-- Minimal bumperbot with two drive wheels and ros2_control mock hardware. -->
 <robot name="bumperbot" xmlns:xacro="http://ros.org/wiki/xacro">
+  <!-- Base footprint (map->base_footprint->base_link) -->
   <link name="base_footprint"/>
+  <!-- Main chassis -->
   <link name="base_link">
     <inertial>
@@ -20,4 +23,5 @@
     </collision>
   </link>
+  <!-- Fixed transform from base_footprint to base_link -->
   <joint name="base_joint" type="fixed">
     <parent link="base_footprint"/>
@@ -25,5 +29,5 @@
     <origin xyz="0 0 0.033" rpy="0 0 0"/>
   </joint>
-  <!-- Wheels as cylinders -->
+  <!-- Right wheel as a cylinder -->
   <link name="wheel_right_link">
     <visual>
@@ -49,5 +53,5 @@
     <axis xyz="0 0 1" />
   </joint>
-  <!-- Left wheel -->
+  <!-- Left wheel as a cylinder -->
   <link name="wheel_left_link">
     <visual>
@@ -73,4 +77,5 @@
     <axis xyz="0 0 1" />
   </joint>
+  <!-- ros2_control mock hardware + interfaces for wheel joints -->
   <ros2_control name="BumperBotSystem" type="system">
     <hardware>
@@ -89,6 +94,5 @@
     </joint>
   </ros2_control>
-  <!-- Comment out gazebo plugin for now -->
-  <!--
+  <!-- Enable Gazebo ros2_control plugin so controllers drive the robot in sim -->
   <gazebo>
     <plugin name="gazebo_ros2_control" filename="libgazebo_ros2_control.so">
@@ -96,4 +100,3 @@
     </plugin>
   </gazebo>
-  -->
 </robot>

Commit message: Restore 2-wheel diff drive and add PlotJuggler docs

File: src/bumperbot_description/urdf/bumperbot.urdf.xacro (robot description, xacro)
@@ -193,3 +193,24 @@
     <axis xyz="0 0 0" />
   </joint>
+  <ros2_control name="BumperBotSystem" type="system">
+    <hardware>
+      <plugin>gz_ros2_control/GazeboSimSystem</plugin>
+    </hardware>
+    <joint name="wheel_right_joint">
+      <command_interface name="velocity"/>
+      <state_interface   name="position"/>
+      <state_interface   name="velocity"/>
+    </joint>
+    <joint name="wheel_left_joint">
+      <command_interface name="velocity"/>
+      <state_interface   name="position"/>
+      <state_interface   name="velocity"/>
+    </joint>
+  </ros2_control>
+  <gazebo>
+    <plugin name="gz_ros2_control::GazeboSimROS2ControlPlugin"
+            filename="gz_ros2_control-system">
+      <parameters>$(find bumperbot_controller)/config/bumperbot_controllers.yaml</parameters>
+    </plugin>
+  </gazebo>
 </robot>

File: src/bumperbot_description/urdf/bumperbot_gazebo.xacro (robot description, xacro)
@@ -13,45 +13,26 @@
     <material>Gazebo/Black</material>
   </gazebo>
-  <gazebo reference="caster_front_link">
-    <material>Gazebo/Red</material>
-  </gazebo>
-  <gazebo reference="caster_rear_link">
-    <material>Gazebo/Red</material>
-  </gazebo>
   <!-- High friction on drive wheels to avoid slipping in simple worlds -->
   <gazebo reference="wheel_right_link">
-    <mu1>1.0</mu1>
-    <mu2>1.0</mu2>
-    <kp>1000000.0</kp>
-    <kd>10.0</kd>
+    <mu1>0.5</mu1>
+    <mu2>0.5</mu2>
+    <kp>500000.0</kp>
+    <kd>5.0</kd>
     <minDepth>0.001</minDepth>
-    <maxVel>0.1</maxVel>
+    <maxVel>0.2</maxVel>
+    <slip1>0.2</slip1>
+    <slip2>0.2</slip2>
     <fdir1>1 0 0</fdir1>
   </gazebo>
   <gazebo reference="wheel_left_link">
-    <mu1>1.0</mu1>
-    <mu2>1.0</mu2>
-    <kp>1000000.0</kp>
-    <kd>10.0</kd>
+    <mu1>0.5</mu1>
+    <mu2>0.5</mu2>
+    <kp>500000.0</kp>
+    <kd>5.0</kd>
     <minDepth>0.001</minDepth>
-    <maxVel>0.1</maxVel>
+    <maxVel>0.2</maxVel>
+    <slip1>0.2</slip1>
+    <slip2>0.2</slip2>
     <fdir1>1 0 0</fdir1>
-  </gazebo>
-  <!-- Lower friction on casters so they slide/rotate easily -->
-  <gazebo reference="caster_front_link">
-    <mu1>0.1</mu1>
-    <mu2>0.1</mu2>
-    <kp>1000000.0</kp>
-    <kd>100.0</kd>
-    <minDepth>0.001</minDepth>
-    <maxVel>0.1</maxVel>
-  </gazebo>
-  <gazebo reference="caster_rear_link">
-    <mu1>0.1</mu1>
-    <mu2>0.1</mu2>
-    <kp>1000000.0</kp>
-    <kd>100.0</kd>
-    <minDepth>0.001</minDepth>
-    <maxVel>0.1</maxVel>
   </gazebo>
   <!-- ROS 2 Control -->
@@ -59,5 +40,5 @@
   <!-- ROS 2 Humble (Ignition) -->
   <xacro:if value="${arg is_ignition}">
-    <plugin filename="ign_ros2_control-system" name="ign_ros2_control::IgnitionROS2ControlPlugin">
+    <plugin filename="gz_ros2_control-system" name="gz_ros2_control::GazeboSimROS2ControlPlugin">
       <parameters>$(find bumperbot_controller)/config/bumperbot_controllers.yaml</parameters>
     </plugin>

File: src/bumperbot_description/urdf/bumperbot_ros2_control.xacro (robot description, xacro)
@@ -3,5 +3,5 @@
   <ros2_control name="BumperBotSystem" type="system">
     <hardware>
-      <plugin>gazebo_ros2_control/GazeboSystem</plugin>
+      <plugin>gz_ros2_control/GazeboSimSystem</plugin>
     </hardware>
     <joint name="wheel_right_joint">
@@ -17,6 +17,6 @@
   </ros2_control>
   <gazebo>
-    <plugin name="gazebo_ros2_control"
-            filename="libgazebo_ros2_control.so">
+    <plugin name="gz_ros2_control::GazeboSimROS2ControlPlugin"
+            filename="gz_ros2_control-system">
       <parameters>
         $(find bumperbot_controller)/config/bumperbot_controllers.yaml
