Commit message: Update bumperbot planning package and workspace

File: src/bumperbot_description/urdf/bumperbot.urdf.xacro (robot description, xacro)
@@ -1,61 +1,12 @@
 <?xml version="1.0"?>
-<!--
-  Bumperbot URDF (xacro): describes a simple differential drive robot base with two drive wheels
-  and two caster wheels. Visuals reference STL meshes packaged under bumperbot_description/meshes.
-  Gazebo classic tags adjust materials and contact properties for reasonable behavior in simulation.
--->
 <robot name="bumperbot" xmlns:xacro="http://ros.org/wiki/xacro">
-  <!-- Gazebo-specific visuals and contact/friction parameters (inlined) -->
-  <gazebo reference="base_link">
-    <material>Gazebo/Blue</material>
-  </gazebo>
-  <gazebo reference="wheel_right_link">
-    <material>Gazebo/Black</material>
-  </gazebo>
-  <gazebo reference="wheel_left_link">
-    <material>Gazebo/Black</material>
-  </gazebo>
-  <gazebo reference="caster_front_link">
-    <material>Gazebo/Red</material>
-  </gazebo>
-  <gazebo reference="caster_rear_link">
-    <material>Gazebo/Red</material>
-  </gazebo>
-  <!-- High friction on drive wheels to avoid slipping in simple worlds -->
-  <gazebo reference="wheel_right_link">
-    <mu1>1.0</mu1>
-    <mu2>1.0</mu2>
-    <kp>1000000.0</kp>
-    <kd>10.0</kd>
-    <minDepth>0.001</minDepth>
-    <maxVel>0.1</maxVel>
-    <fdir1>1 0 0</fdir1>
-  </gazebo>
-  <gazebo reference="wheel_left_link">
-    <mu1>1.0</mu1>
-    <mu2>1.0</mu2>
-    <kp>1000000.0</kp>
-    <kd>10.0</kd>
-    <minDepth>0.001</minDepth>
-    <maxVel>0.1</maxVel>
-    <fdir1>1 0 0</fdir1>
-  </gazebo>
-  <!-- Lower friction on casters so they slide/rotate easily -->
-  <gazebo reference="caster_front_link">
-    <mu1>0.1</mu1>
-    <mu2>0.1</mu2>
-    <kp>1000000.0</kp>
-    <kd>100.0</kd>
-    <minDepth>0.001</minDepth>
-    <maxVel>0.1</maxVel>
-  </gazebo>
-  <gazebo reference="caster_rear_link">
-    <mu1>0.1</mu1>
-    <mu2>0.1</mu2>
-    <kp>1000000.0</kp>
-    <kd>100.0</kd>
-    <minDepth>0.001</minDepth>
-    <maxVel>0.1</maxVel>
-  </gazebo>
+  <!-- Start GZ or Ignition depending on ROS 2 Version -->
+  <xacro:arg name="is_ignition" default="true"/>
+  <!-- Load Simulated or Real Hardware Interfaces -->
+  <xacro:arg name="is_sim" default="true"/>
+  <!-- Include Gazebo Parameters -->
+  <xacro:include filename="$(find bumperbot_description)/urdf/bumperbot_gazebo.xacro" />
+  <!-- Include ros2_control Plugins -->
+  <xacro:include filename="$(find bumperbot_description)/urdf/bumperbot_ros2_control.xacro" />
   <link name="base_footprint"/>
   <link name="base_link">
@@ -72,4 +23,5 @@
         <mesh filename="package://bumperbot_description/meshes/base_link.STL" />
       </geometry>
+      <material name="black"/>
     </visual>
     <collision>
@@ -98,4 +50,5 @@
         <mesh filename="package://bumperbot_description/meshes/wheel_right_link.STL" />
       </geometry>
+      <material name="blue"/>
     </visual>
     <collision>
@@ -112,5 +65,6 @@
     <axis xyz="0 1 0" />
   </joint>
-  <link name="wheel_left_link">
+  <link
+    name="wheel_left_link">
     <inertial>
       <origin xyz="0 0.014 0" rpy="0 0 0" />
@@ -125,4 +79,5 @@
         <mesh filename="package://bumperbot_description/meshes/wheel_left_link.STL" />
       </geometry>
+      <material name="blue"/>
     </visual>
     <collision>
@@ -152,4 +107,5 @@
         <mesh filename="package://bumperbot_description/meshes/caster_front_link.STL" />
       </geometry>
+      <material name="silver"/>
     </visual>
     <collision>
@@ -179,4 +135,5 @@
         <mesh filename="package://bumperbot_description/meshes/caster_rear_link.STL" />
       </geometry>
+      <material name="silver"/>
     </visual>
     <collision>
@@ -193,24 +150,71 @@
     <axis xyz="0 0 0" />
   </joint>
-  <ros2_control name="BumperBotSystem" type="system">
-    <hardware>
-      <plugin>gz_ros2_control/GazeboSimSystem</plugin>
-    </hardware>
-    <joint name="wheel_right_joint">
-      <command_interface name="velocity"/>
-      <state_interface   name="position"/>
-      <state_interface   name="velocity"/>
-    </joint>
-    <joint name="wheel_left_joint">
-      <command_interface name="velocity"/>
-      <state_interface   name="position"/>
-      <state_interface   name="velocity"/>
-    </joint>
-  </ros2_control>
-  <gazebo>
-    <plugin name="gz_ros2_control::GazeboSimROS2ControlPlugin"
-            filename="gz_ros2_control-system">
-      <parameters>$(find bumperbot_controller)/config/bumperbot_controllers.yaml</parameters>
-    </plugin>
-  </gazebo>
+  <link name="imu_link">
+    <inertial>
+      <origin xyz="-0.00552433659106688 0.000168210391520346 0.000514000497342681" rpy="0 0 0" />
+      <mass value="0.000528415362211671" />
+      <inertia ixx="1.46176048428261E-08" ixy="1.40015117949421E-10" ixz="-1.99633872937403E-12"
+               iyy="8.59662482954888E-09" iyz="7.52375112767959E-12"
+               izz="2.30279421279312E-08" />
+    </inertial>
+    <visual>
+      <origin xyz="0 0 0" rpy="0 0 0" />
+      <geometry>
+        <mesh filename="package://bumperbot_description/meshes/imu_link.STL" />
+      </geometry>
+      <material name="blue"/>
+    </visual>
+    <collision>
+      <origin xyz="0 0 0" rpy="0 0 0" />
+      <geometry>
+        <mesh filename="package://bumperbot_description/meshes/imu_link.STL" />
+      </geometry>
+    </collision>
+  </link>
+  <joint name="imu_joint" type="fixed">
+    <origin xyz="0 0 0.0698986241758014" rpy="0 0 0" />
+    <parent link="base_link" />
+    <child link="imu_link" />
+    <axis xyz="0 0 0" />
+  </joint>
+  <link name="laser_link">
+    <inertial>
+      <origin xyz="-0.011945780406062 -0.000381929217680526 -0.0170649378129477" rpy="0 0 0" />
+      <mass value="0.073084435549317" />
+      <inertia ixx="1.96074931730795E-05" ixy="-3.62091076640009E-07" ixz="4.28230084046735E-07"
+               iyy="2.40983835136327E-05" iyz="1.50180909250652E-08"
+               izz="4.14184164228595E-05" />
+    </inertial>
+    <visual>
+      <origin xyz="0 0 0" rpy="0 0 0" />
+      <geometry>
+        <mesh filename="package://bumperbot_description/meshes/laser_link.STL" />
+      </geometry>
+      <material name="dark_grey"/>
+    </visual>
+    <collision>
+      <origin xyz="0 0 0" rpy="0 0 0" />
+      <geometry>
+        <mesh filename="package://bumperbot_description/meshes/laser_link.STL" />
+      </geometry>
+    </collision>
+  </link>
+  <joint name="laser_joint" type="fixed">
+    <origin xyz="-0.0050526 -0.0023221 0.1208" rpy="0 0 3.14" />
+    <parent link="base_link" />
+    <child link="laser_link" />
+    <axis xyz="0 0 0" />
+  </joint>
+  <material name="blue">
+    <color rgba="0 0 1 1"/>
+  </material>
+  <material name="black">
+    <color rgba="0 0 0 1"/>
+  </material>
+  <material name="silver">
+    <color rgba="0.79 0.82 0.93 1"/>
+  </material>
+  <material name="dark_grey">
+    <color rgba="0.3 0.3 0.3 1"/>
+  </material>
 </robot>

File: src/bumperbot_description/urdf/bumperbot_gazebo.xacro (robot description, xacro)
@@ -1,107 +1,145 @@
 <?xml version="1.0"?>
-<!-- Gazebo-specific visuals and contact/friction parameters.
-     This file is included by xacro; do not wrap in a <robot> tag. -->
-<xacro:macro name="bumperbot_gazebo_props" xmlns:xacro="http://ros.org/wiki/xacro">
-  <!-- Colors for quick visual identification -->
-  <gazebo reference="base_link">
-    <material>Gazebo/Blue</material>
+<robot name="bumperbot" xmlns:xacro="http://ros.org/wiki/xacro">
+  <!-- Wheels -->
+  <gazebo reference="wheel_left_link">
+    <mu1>1000000000000000.0</mu1>
+    <mu2>1000000000000000.0</mu2>
+    <kp>1000000000000.0</kp>
+    <kd>10.0</kd>
+    <minDepth>0.001</minDepth>
+    <maxVel>0.1</maxVel>
+    <fdir1>1 0 0</fdir1>
   </gazebo>
   <gazebo reference="wheel_right_link">
-    <material>Gazebo/Black</material>
-  </gazebo>
-  <gazebo reference="wheel_left_link">
-    <material>Gazebo/Black</material>
-  </gazebo>
-  <!-- High friction on drive wheels to avoid slipping in simple worlds -->
-  <gazebo reference="wheel_right_link">
-    <mu1>0.5</mu1>
-    <mu2>0.5</mu2>
-    <kp>500000.0</kp>
-    <kd>5.0</kd>
+    <mu1>1000000000000000.0</mu1>
+    <mu2>1000000000000000.0</mu2>
+    <kp>1000000000000.0</kp>
+    <kd>10.0</kd>
     <minDepth>0.001</minDepth>
-    <maxVel>0.2</maxVel>
-    <slip1>0.2</slip1>
-    <slip2>0.2</slip2>
+    <maxVel>0.1</maxVel>
     <fdir1>1 0 0</fdir1>
   </gazebo>
-  <gazebo reference="wheel_left_link">
-    <mu1>0.5</mu1>
-    <mu2>0.5</mu2>
-    <kp>500000.0</kp>
-    <kd>5.0</kd>
+  <!-- Caster Wheels -->
+  <gazebo reference="caster_rear_link">
+    <mu1>0.1</mu1>
+    <mu2>0.1</mu2>
+    <kp>1000000.0</kp>
+    <kd>100.0</kd>
     <minDepth>0.001</minDepth>
-    <maxVel>0.2</maxVel>
-    <slip1>0.2</slip1>
-    <slip2>0.2</slip2>
-    <fdir1>1 0 0</fdir1>
+    <maxVel>1.0</maxVel>
+  </gazebo>
+  <gazebo reference="caster_front_link">
+    <mu1>0.1</mu1>
+    <mu2>0.1</mu2>
+    <kp>1000000.0</kp>
+    <kd>100.0</kd>
+    <minDepth>0.001</minDepth>
+    <maxVel>1.0</maxVel>
   </gazebo>
   <!-- ROS 2 Control -->
-<gazebo>
-  <!-- ROS 2 Humble (Ignition) -->
-  <xacro:if value="${arg is_ignition}">
-    <plugin filename="gz_ros2_control-system" name="gz_ros2_control::GazeboSimROS2ControlPlugin">
-      <parameters>$(find bumperbot_controller)/config/bumperbot_controllers.yaml</parameters>
-    </plugin>
-    <plugin filename="ignition-gazebo-imu-system" name="ignition::gazebo::systems::Imu"/>
-  </xacro:if>
-  <!-- ROS 2 Iron or above (Gazebo / ros_gz_sim) -->
-  <xacro:unless value="${arg is_ignition}">
-    <plugin filename="gz_ros2_control-system" name="gz_ros2_control::GazeboSimROS2ControlPlugin">
-      <parameters>$(find bumperbot_controller)/config/bumperbot_controllers.yaml</parameters>
-    </plugin>
-    <plugin filename="gz-sim-imu-system" name="gz::sim::systems::Imu"/>
-  </xacro:unless>
-</gazebo>
-<gazebo reference="imu_link">
-  <sensor name="imu" type="imu">
-    <always_on>true</always_on>
-    <update_rate>100</update_rate>
-    <gz_frame_id>imu_link</gz_frame_id>
-    <topic>imu</topic>
-    <imu>
-      <!-- Angular velocity noise -->
-      <angular_velocity>
-        <x>
-          <noise type="gaussian">
-            <mean>0.0</mean>
-            <stddev>2e-4</stddev>
-          </noise>
-        </x>
-        <y>
-          <noise type="gaussian">
-            <mean>0.0</mean>
-            <stddev>2e-4</stddev>
-          </noise>
-        </y>
-        <z>
-          <noise type="gaussian">
-            <mean>0.0</mean>
-            <stddev>2e-4</stddev>
-          </noise>
-        </z>
-      </angular_velocity>
-      <!-- Linear acceleration noise -->
-      <linear_acceleration>
-        <x>
-          <noise type="gaussian">
-            <mean>0.0</mean>
-            <stddev>1.7e-2</stddev>
-          </noise>
-        </x>
-        <y>
-          <noise type="gaussian">
-            <mean>0.0</mean>
-            <stddev>1.7e-2</stddev>
-          </noise>
-        </y>
-        <z>
-          <noise type="gaussian">
-            <mean>0.0</mean>
-            <stddev>1.7e-2</stddev>
-          </noise>
-        </z>
-      </linear_acceleration>
-    </imu>
-  </sensor>
-</gazebo>
-</xacro:macro>
+  <gazebo>
+    <!-- ROS 2 Humble -->
+    <xacro:if value="$(arg is_ignition)">
+      <plugin filename="ign_ros2_control-system" name="ign_ros2_control::IgnitionROS2ControlPlugin">
+        <parameters>$(find bumperbot_controller)/config/bumperbot_controllers.yaml</parameters>
+      </plugin>
+      <plugin filename="ignition-gazebo-imu-system" name="ignition::gazebo::systems::Imu">
+      </plugin>
+      <plugin filename="ignition-gazebo-sensors-system" name="ignition::gazebo::systems::Sensors">
+        <render_engine>ogre2</render_engine>
+      </plugin>
+    </xacro:if>
+    <!-- ROS 2 Iron or above -->
+    <xacro:unless value="$(arg is_ignition)">
+      <plugin filename="gz_ros2_control-system" name="gz_ros2_control::GazeboSimROS2ControlPlugin">
+        <parameters>$(find bumperbot_controller)/config/bumperbot_controllers.yaml</parameters>
+      </plugin>
+      <plugin filename="gz-sim-imu-system" name="gz::sim::systems::Imu">
+      </plugin>
+      <plugin filename="gz-sim-sensors-system" name="gz::sim::systems::Sensors">
+        <render_engine>ogre2</render_engine>
+      </plugin>
+    </xacro:unless>
+  </gazebo>
+  <!-- IMU -->
+  <gazebo reference="imu_link">
+    <sensor name="imu" type="imu">
+        <always_on>true</always_on>
+        <update_rate>100</update_rate>
+        <gz_frame_id>imu_link</gz_frame_id>
+        <topic>imu</topic>
+        <imu>
+          <angular_velocity>
+            <x>
+              <noise type="gaussian">
+                <mean>0.0</mean>
+                <stddev>2e-4</stddev>
+              </noise>
+            </x>
+            <y>
+              <noise type="gaussian">
+                <mean>0.0</mean>
+                <stddev>2e-4</stddev>
+              </noise>
+            </y>
+            <z>
+              <noise type="gaussian">
+                <mean>0.0</mean>
+                <stddev>2e-4</stddev>
+              </noise>
+            </z>
+          </angular_velocity>
+          <linear_acceleration>
+            <x>
+              <noise type="gaussian">
+                <mean>0.0</mean>
+                <stddev>1.7e-2</stddev>
+              </noise>
+            </x>
+            <y>
+              <noise type="gaussian">
+                <mean>0.0</mean>
+                <stddev>1.7e-2</stddev>
+              </noise>
+            </y>
+            <z>
+              <noise type="gaussian">
+                <mean>0.0</mean>
+                <stddev>1.7e-2</stddev>
+              </noise>
+            </z>
+          </linear_acceleration>
+        </imu>
+    </sensor>
+  </gazebo>
+  <!-- 2D Laser Sensor -->
+  <gazebo reference="laser_link">
+    <sensor name="lidar" type="gpu_lidar">
+      <always_on>true</always_on>
+      <visualize>true</visualize>
+      <topic>scan</topic>
+      <update_rate>5</update_rate>
+      <gz_frame_id>laser_link</gz_frame_id>
+      <lidar>
+        <scan>
+          <horizontal>
+            <samples>360</samples>
+            <resolution>1.00000</resolution>
+            <min_angle>0.000000</min_angle>
+            <max_angle>6.280000</max_angle>
+          </horizontal>
+        </scan>
+        <range>
+          <min>0.120000</min>
+          <max>12.0</max>
+          <resolution>0.02</resolution>
+        </range>
+        <noise>
+          <type>gaussian</type>
+          <mean>0.0</mean>
+          <stddev>0.01</stddev>
+        </noise>
+      </lidar>
+    </sensor>
+  </gazebo>
+</robot>

File: src/bumperbot_description/urdf/bumperbot_ros2_control.xacro (robot description, xacro)
@@ -1,26 +1,44 @@
 <?xml version="1.0"?>
-<robot xmlns:xacro="http://ros.org/wiki/xacro">
-  <ros2_control name="BumperBotSystem" type="system">
-    <hardware>
-      <plugin>gz_ros2_control/GazeboSimSystem</plugin>
-    </hardware>
-    <joint name="wheel_right_joint">
-      <command_interface name="velocity"/>
-      <state_interface   name="position"/>
-      <state_interface   name="velocity"/>
-    </joint>
-    <joint name="wheel_left_joint">
-      <command_interface name="velocity"/>
-      <state_interface   name="position"/>
-      <state_interface   name="velocity"/>
-    </joint>
-  </ros2_control>
-  <gazebo>
-    <plugin name="gz_ros2_control::GazeboSimROS2ControlPlugin"
-            filename="gz_ros2_control-system">
-      <parameters>
-        $(find bumperbot_controller)/config/bumperbot_controllers.yaml
-      </parameters>
-    </plugin>
-  </gazebo>
+<robot xmlns:xacro="http://www.ros.org/wiki/xacro" name="bumperbot">
+    <ros2_control name="RobotSystem" type="system">
+        <!-- ros2_control Gazebo -->
+        <xacro:if value="$(arg is_sim)">
+            <!-- ROS 2 Humble -->
+            <xacro:if value="$(arg is_ignition)">
+                <hardware>
+                    <plugin>ign_ros2_control/IgnitionSystem</plugin>
+                </hardware>
+            </xacro:if>
+            <!-- ROS 2 Iron or above -->
+            <xacro:unless value="$(arg is_ignition)">
+                <hardware>
+                    <plugin>gz_ros2_control/GazeboSimSystem</plugin>
+                </hardware>
+            </xacro:unless>
+        </xacro:if>
+        <!-- ros2_control Real Robot -->
+        <xacro:unless value="$(arg is_sim)">
+            <hardware>
+                <plugin>bumperbot_firmware/BumperbotInterface</plugin>
+                <param name="port">/dev/ttyUSB0</param>
+            </hardware>
+        </xacro:unless>
+        <!-- ros2_control Common Interfaces -->
+        <joint name="wheel_left_joint">
+            <command_interface name="velocity">
+              <param name="min">-1</param>
+              <param name="max">1</param>
+            </command_interface>
+            <state_interface name="position" />
+            <state_interface name="velocity" />
+        </joint>
+        <joint name="wheel_right_joint">
+            <command_interface name="velocity">
+              <param name="min">-1</param>
+              <param name="max">1</param>
+            </command_interface>
+            <state_interface name="position" />
+            <state_interface name="velocity" />
+        </joint>
+    </ros2_control>
 </robot>
